File: Motw.kicad_sch (KiCad schematic)
At the start: 110 parts, among them J1 Barrel_Jack_Switch, J2 AudioJack3, J3 AudioJack2, Q1 2SC2240, Q14 2SC2240, Q18 2SC2240, Q3 2SC2240, Q4 2SA970, Q5 2SK30A, U1 TL072, U2 TL074

Commit message: v2.0.0
Parts:
- removed C10: 10u, Capacitor_THT:CP_Radial_D5.0mm_P2.00mm, symbol Device:C_Polarized
- removed C13, C37, C38: 10u, Capacitor_THT:CP_Radial_D5.0mm_P2.00mm, symbol Device:C_Polarized_Small
- removed C16: 1u, Capacitor_THT:CP_Radial_D5.0mm_P2.00mm, symbol Device:C_Polarized
- removed C19: 68n, Capacitor_THT:C_Rect_L8.5mm_W5.5mm_P5.00mm_FKS2_FKP2_MKS2_MKP2, symbol Device:C
- removed C27: 47n, Capacitor_THT:C_Rect_L8.5mm_W5.5mm_P5.00mm_FKS2_FKP2_MKS2_MKP2, symbol Device:C
- removed C7: 1.5u, Capacitor_THT:C_Rect_L7.2mm_W5.5mm_P5.00mm_FKS2_FKP2_MKS2_MKP2, symbol Device:C
- removed C9: 100p, Capacitor_THT:C_Rect_L7.0mm_W2.5mm_P5.00mm, symbol Device:C
- removed Q14: 2SC2240, Package_TO_SOT_THT:TO-92_231, symbol Device:Q_NPN_BEC
- removed Q3: 2SC2240, Package_TO_SOT_THT:TO-92_231, symbol Simulation_SPICE:NPN
- removed Q4: 2SA970, Package_TO_SOT_THT:TO-92_231, symbol Simulation_SPICE:PNP
- removed R27: 4.7k, Resistor_THT:R_Axial_DIN0207_L6.3mm_D2.5mm_P7.62mm_Horizontal, symbol Device:R_Small
- removed R31: 10k, Resistor_THT:R_Axial_DIN0207_L6.3mm_D2.5mm_P7.62mm_Horizontal, symbol Device:R_Small
- removed R32: 1k, Resistor_THT:R_Axial_DIN0207_L6.3mm_D2.5mm_P7.62mm_Horizontal, symbol Device:R_Small
- removed R33, R73: 100k, Resistor_THT:R_Axial_DIN0207_L6.3mm_D2.5mm_P7.62mm_Horizontal, symbol Device:R_Small
- removed VR3: 10k, Potentiometer_THT:Potentiometer_RD9, symbol Device:R_Potentiometer_Small
- added C10: 180n, Capacitor_THT:C_Rect_L8.5mm_W5.5mm_P5.00mm_FKS2_FKP2_MKS2_MKP2, symbol Device:C
- added C13: 100p, Capacitor_THT:C_Rect_L7.0mm_W2.5mm_P5.00mm, symbol Device:C
- added C16: 4.7n, Capacitor_THT:C_Rect_L6.5mm_W3.5mm_P3.50mm_MKS02_FKP02, symbol Device:C
- added C19: 1u, Capacitor_THT:CP_Radial_D5.0mm_P2.00mm, symbol Device:C_Polarized
- added C23: 470p, Capacitor_THT:C_Rect_L7.0mm_W2.5mm_P5.00mm, symbol Device:C
- added C27, C28, C9: 10u, Capacitor_THT:CP_Radial_D5.0mm_P2.00mm, symbol Device:C_Polarized
- added C7: 47u, Capacitor_THT:CP_Radial_D8.0mm_P3.50mm, symbol Device:C_Polarized
- added Q2: 2SC2240, Package_TO_SOT_THT:TO-92_231, symbol Simulation_SPICE:NPN
- added Q3: 2SA970, Package_TO_SOT_THT:TO-92_231, symbol Simulation_SPICE:PNP
- added Q4: 2SC2240, Package_TO_SOT_THT:TO-92_231, symbol Device:Q_NPN_BEC
- added R27: 330, Resistor_THT:R_Axial_DIN0207_L6.3mm_D2.5mm_P7.62mm_Horizontal, symbol Device:R
- added R31: 4.7k, Resistor_THT:R_Axial_DIN0207_L6.3mm_D2.5mm_P7.62mm_Horizontal, symbol Device:R
- added R32: 100k, Resistor_THT:R_Axial_DIN0207_L6.3mm_D2.5mm_P7.62mm_Horizontal, symbol Device:R
- added R33: 10k, Resistor_THT:R_Axial_DIN0207_L6.3mm_D2.5mm_P7.62mm_Horizontal, symbol Device:R
- added R35: 1k, Resistor_THT:R_Axial_DIN0207_L6.3mm_D2.5mm_P7.62mm_Horizontal, symbol Device:R
- added VR1: 10k, Potentiometer_THT:Potentiometer_RD9, symbol Device:R_Potentiometer
- C1, C2, C26, C5: symbol Device:C_Polarized_Small -> Device:C_Polarized
- C11: value 47n -> 100p; footprint Capacitor_THT:C_Rect_L8.5mm_W5.5mm_P5.00mm_FKS2_FKP2_MKS2_MKP2 -> Capacitor_THT:C_Rect_L7.0mm_W2.5mm_P5.00mm
- C12: value 100p -> 47n; footprint Capacitor_THT:C_Rect_L7.0mm_W2.5mm_P5.00mm -> Capacitor_THT:C_Rect_L8.5mm_W5.5mm_P5.00mm_FKS2_FKP2_MKS2_MKP2
- C15: value 1n -> 68n; footprint Capacitor_THT:C_Rect_L6.0mm_W3.0mm_P3.50mm_MKS02_FKP02 -> Capacitor_THT:C_Rect_L8.5mm_W5.5mm_P5.00mm_FKS2_FKP2_MKS2_MKP2
- C17: value 470p -> 6.8n; footprint Capacitor_THT:C_Rect_L7.0mm_W2.5mm_P5.00mm -> Capacitor_THT:C_Rect_L6.5mm_W3.5mm_P3.50mm_MKS02_FKP02
- C18: value 0.1u -> 1n; footprint Capacitor_THT:C_Rect_L7.5mm_W3.0mm_P5.00mm -> Capacitor_THT:C_Rect_L6.0mm_W3.0mm_P3.50mm_MKS02_FKP02
- C20: value 4.7n -> 1.5u; footprint Capacitor_THT:C_Rect_L6.5mm_W3.5mm_P3.50mm_MKS02_FKP02 -> Capacitor_THT:C_Rect_L7.2mm_W5.5mm_P5.00mm_FKS2_FKP2_MKS2_MKP2
- C21: value 0.15u -> 0.1u
- C22: value 6.8n -> 0.15u; footprint Capacitor_THT:C_Rect_L6.5mm_W3.5mm_P3.50mm_MKS02_FKP02 -> Capacitor_THT:C_Rect_L7.5mm_W3.0mm_P5.00mm
- C24: value 47u -> 10u; footprint Capacitor_THT:CP_Radial_D8.0mm_P3.50mm -> Capacitor_THT:CP_Radial_D5.0mm_P2.00mm
- C25, C3, C4: symbol Device:C_Small -> Device:C
- C6: value 47n -> 180n
- D2: symbol Device:D_Zener_Small -> Device:D_Zener
- R1, R2, R48, R49, R5, R50, R51, R52, R6: symbol Device:R_Small -> Device:R
- R10: value 150 -> 22
- R11: value 22k -> 150
- R12, R4: value 100k -> 22k
- R13: value 120 -> 100k
- R15: value 10k -> 120
- R16: value 47k -> 10k
- R17: value 220k -> 68k
- R18: value 10k -> 47k
- R19: value 10k -> 220k
- R20: value 3.3k -> 10k
- R21: value 3.3k -> 100k
- R22: value 330 -> 100k
- R23: value 100k -> 82k
- R24: value 100k -> 10k
- R26: value 82k -> 330
- R28: value 330 -> 68k
- R29, R30: value 68k -> 3.3k
- R3: value 22k -> 1k
- R34: value 1k -> 100k
- R7: value 470k -> 100k
- R8: value 10k -> 470k
- R9: value 22 -> 10k
Connections:
- net +4V: now also R21.1, R22.1, R28.2, R32.2, VR1.1; no longer R24.1, R26.1, R30.2
- net +8V: now also R17.2, R3.1, Q4.3 (C); no longer R29.2, R34.1
- net GND: now also C18.2, R10.1, R16.1, R34.2, R7.1, C7.2, R33.2; no longer C15.2, C24.2, R15.1, R4.1, R9.1
- net at RV1.1: now also R11.1; no longer R10.1
- net at R10.2: now also Q2.3 (E)
- net at R9.2: now also R13.2, R15.2, R3.2, C7.1
- net at U1.5 (+): now also R28.1, C19.2; no longer R30.1
- net at D10.2 (A), D11.1 (K): now also C18.1, R24.2, C19.1; no longer C15.1, R19.2
- net at C12.1, D5.1 (K), U1.2 (-): now also D6.2 (A), R19.1, C13.1; no longer C11.1, D7.2 (A), R17.1
- net at R14.2, U1.3 (+): now also C11.2, R16.2, R17.1, Q3.1 (C); no longer R15.2, R29.1
- net at RV1.3: now also R18.1; no longer R16.1
- net at C21.2, RV3.2: now also C22.2; no longer C18.2
- net at U2.13 (-), U2.14: now also R27.1; no longer R28.1
- net at C14.2: now also R20.1; no longer R18.1
- net at R13.1: now also C11.1, R12.2, R14.1, Q3.2 (B)
- net at H14.1: now also R35.2; no longer J3.T
- net at R7.2, R8.1: now also C8.1, R4.2, Q2.2 (B); no longer C6.1, C8.2
- net at C6.2: now also R4.1; no longer R11.1
- net at R22.2: now also U2.10 (+), C16.1
- net at RV2.2: now also C20.2
- net at U2.6 (-), U2.7: now also R25.1; no longer R22.1
- net at U2.8, U2.9 (-): now also R26.1; no longer R25.1
- net at D8.2 (A), D9.1 (K): now also R24.1; no longer R19.1
- net at D8.1 (K), D9.2 (A): now also R20.2; no longer R18.2
- net at Q18.3 (C), Q5.3 (S): now also C6.1
- net at H15.1: now also J3.T
- net at U1.6 (-), U1.7: now also R29.1; no longer R21.1
- net at RV2.1, RV3.1, U2.3 (+): now also R29.2; no longer R21.2
- net at RV2.3, RV3.3, U2.2 (-): now also R30.1, C23.1; no longer C17.1, R20.1
- net at D5.2 (A): now also D7.1 (K); no longer D6.1 (K)
- net at R23.2: now also C17.1, U2.12 (+); no longer U2.5 (+)
- new net: C28.2, R34.1, R35.1
- new net: C10.1, C8.2, C9.1, Q2.1 (C), R8.2, R9.1
- new net: C9.2, R11.2
- new net: Q3.3 (E), R15.1
- new net: C10.2, R12.1
- new net: C27.2, Q4.1 (B), R32.1
- new net: C28.1, Q4.2 (E), R33.1
- new net: C16.2, C21.1, R26.2
- new net: C27.1, VR1.2
- new net: R31.1, VR1.3
- new net: C13.2, C14.1, D6.1 (K), D7.2 (A), R19.2, U1.1
- new net: C12.2, R18.2
- new net: C23.2, C24.1, R30.2, U2.1
- new net: C15.2, C20.1, R25.2
- new net: C17.2, C22.1, R27.2
- new net: C15.1, R21.2, U2.5 (+)
- new net: C24.2, R31.2
Other:
- note removed: "LEVEL"
- moved on the sheet: A1, C1, C2, C25, C26, C3, C4, C5, D1, D2, D3, D4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
